Commit message: Adjusting for new hat

File: src/start_creating_robots/worlds_and_models/krytn/krytn.urdf.xacro (robot description, xacro)
@@ -1,8 +1,8 @@
 <?xml version='1.0' encoding='utf-8'?>
-<robot xmlns:xacro="http://www.ros.org/wiki/xacro" name="krytn" >
+<robot xmlns:xacro="http://www.ros.org/wiki/xacro" name="krytn">
     <xacro:arg name="with_sensors" default="true" />
     <!-- Include the robot base. Configure it with a differential drive control plugin -->
     <xacro:include filename="$(find start_creating_robots)/worlds_and_models/krytn/magni.urdf.xacro" />
-    <xacro:if value="$(arg with_sensors)" >
+    <xacro:if value="$(arg with_sensors)">
         <!-- Include an extra 2D Lidar -->
         <xacro:include filename="$(find start_creating_robots)/worlds_and_models/krytn/lidar_2d_v1.urdf.xacro" />
@@ -10,37 +10,45 @@
         <xacro:include filename="$(find start_creating_robots)/worlds_and_models/krytn/realsense_d435.urdf.xacro" />
     </xacro:if>
+    <xacro:if value="True">
+        <link name="krytn_top">
+            <visual name="visual">
+                <geometry>
+                    <mesh filename="file://$(find start_creating_robots)/worlds_and_models/krytn/meshes/krytn_top-part.dae"/>
+                </geometry>
+            </visual>
+        </link>
+        <joint name="krytn_top_joint" type="fixed">
+            <parent link="base_footprint" />
+            <child link="krytn_top" />
+            <origin xyz="0.05 0 0.26" rpy="0 0 1.57" />
+        </joint>
+    </xacro:if>
     <!-- Gazebo specific plugins-->
     <gazebo >
-        <xacro:if value="$(arg with_sensors)" >
-            <plugin
-            filename="ignition-gazebo-sensors-system"
-            name="ignition::gazebo::systems::Sensors">
+        <xacro:if value="$(arg with_sensors)">
+            <plugin filename="ignition-gazebo-sensors-system" name="ignition::gazebo::systems::Sensors">
                 <render_engine>ogre2</render_engine>
             </plugin>
         </xacro:if>
         <!-- Publish joints for robot description tf publisher. -->
-        <plugin
-            filename="ignition-gazebo-joint-state-publisher-system"
-            name="ignition::gazebo::systems::JointStatePublisher">
+        <plugin filename="ignition-gazebo-joint-state-publisher-system" name="ignition::gazebo::systems::JointStatePublisher">
             <topic>joint_states</topic>
         </plugin>
         <!-- Plugin to allow Gazebo to recieve cmd_vel and rotate wheels in Gazebo. -->
-        <plugin
-                filename="ignition-gazebo-diff-drive-system"
-                name="ignition::gazebo::systems::DiffDrive">
-                <left_joint>left_wheel_joint</left_joint>
-                <right_joint>right_wheel_joint</right_joint>
-                <frame_id>odom</frame_id>
-                <wheel_separation>0.326</wheel_separation>
-                <wheel_radius>0.128</wheel_radius>
-                <odom_publish_frequency>20</odom_publish_frequency>
-                <max_linear_acceleration>1</max_linear_acceleration>
-                <min_linear_acceleration>-1</min_linear_acceleration>
-                <max_angular_acceleration>2</max_angular_acceleration>
-                <min_angular_acceleration>-2</min_angular_acceleration>
-                <max_linear_velocity>0.5</max_linear_velocity>
-                <min_linear_velocity>-0.5</min_linear_velocity>
-                <max_angular_velocity>1</max_angular_velocity>
-                <min_angular_velocity>-1</min_angular_velocity>
+        <plugin filename="ignition-gazebo-diff-drive-system" name="ignition::gazebo::systems::DiffDrive">
+            <left_joint>left_wheel_joint</left_joint>
+            <right_joint>right_wheel_joint</right_joint>
+            <frame_id>odom</frame_id>
+            <wheel_separation>0.326</wheel_separation>
+            <wheel_radius>0.128</wheel_radius>
+            <odom_publish_frequency>20</odom_publish_frequency>
+            <max_linear_acceleration>1</max_linear_acceleration>
+            <min_linear_acceleration>-1</min_linear_acceleration>
+            <max_angular_acceleration>2</max_angular_acceleration>
+            <min_angular_acceleration>-2</min_angular_acceleration>
+            <max_linear_velocity>0.5</max_linear_velocity>
+            <min_linear_velocity>-0.5</min_linear_velocity>
+            <max_angular_velocity>1</max_angular_velocity>
+            <min_angular_velocity>-1</min_angular_velocity>
         </plugin>
     </gazebo>

File: src/start_creating_robots/worlds_and_models/krytn/lidar_2d_v1.urdf.xacro (robot description, xacro)
@@ -1,63 +1,63 @@
 <?xml version="1.0" ?>
 <robot xmlns:xacro="http://wiki.ros.org/xacro">
-<link name="lidar_2d_v1">
-  <origin xyz="0.1 0 0.36" rpy="0 0 0" />
-  <xacro:cylinder_inertial_with_origin radius="0.02" length="0.35" mass="0.13">
-    <origin xyz="0 0 0.03" rpy="0 ${pi/2} 0" />
-  </xacro:cylinder_inertial_with_origin>
-  <collision name="collision_base">
-    <pose>0 0 0.0175015175 0 0 0</pose>
-    <geometry>
-      <box size="0.05001062 0.05001062 0.035003035"/>
-    </geometry>
-  </collision>
-  <collision name="collision_top">
-    <pose>0 0 0.0525045525 0 0 0</pose>
-    <geometry>
-      <cylinder radius="0.02" length="0.035003035" />
-    </geometry>
-  </collision>
-  <visual name="visual">
-    <pose>0 0 0 0 0 1.5707</pose>
-    <geometry>
-      <mesh filename="file://$(find start_creating_robots)/worlds_and_models/krytn//meshes/lidar_2d_v1.dae"/>
-    </geometry>
-  </visual>
-</link>
-<!-- This joint connects the robot to the lidar -->
-<joint name="lidar_joint" type="fixed">
+  <link name="lidar_2d_v1">
+    <origin xyz="0.1 0 0.36" rpy="0 0 0" />
+    <xacro:cylinder_inertial_with_origin radius="0.02" length="0.35" mass="0.13">
+      <origin xyz="0 0 0.03" rpy="0 ${pi/2} 0" />
+    </xacro:cylinder_inertial_with_origin>
+    <collision name="collision_base">
+      <pose>0 0 0.0175015175 0 0 0</pose>
+      <geometry>
+        <box size="0.05001062 0.05001062 0.035003035"/>
+      </geometry>
+    </collision>
+    <collision name="collision_top">
+      <pose>0 0 0.0525045525 0 0 0</pose>
+      <geometry>
+        <cylinder radius="0.02" length="0.035003035" />
+      </geometry>
+    </collision>
+    <visual name="visual">
+      <pose>0 0 0 0 0 1.5707</pose>
+      <geometry>
+        <mesh filename="file://$(find start_creating_robots)/worlds_and_models/krytn//meshes/lidar_2d_v1.dae"/>
+      </geometry>
+    </visual>
+  </link>
+  <!-- This joint connects the robot to the lidar -->
+  <joint name="lidar_joint" type="fixed">
     <parent link="base_footprint" />
     <child link="lidar_2d_v1" />
-    <origin rpy="0 0 0" xyz="0 0 0.398"/>
-</joint>
-<gazebo reference="lidar_2d_v1">
-  <sensor name="lidar_2d_v1" type="gpu_ray">
-    <topic>lidar</topic>
-    <ignition_frame_id>lidar_2d_v1</ignition_frame_id>
-    <pose>0 0 0.0525045525 0 0 0</pose>
-    <ray>
-      <scan>
-        <horizontal>
-          <samples>90</samples>
-          <resolution>1</resolution>
-          <min_angle>-1.41</min_angle>
-          <max_angle>1.41</max_angle>
-        </horizontal>
-      </scan>
-      <range>
-        <min>0.060</min>
-        <max>10</max>
-        <resolution>0.04</resolution>
-      </range>
-      <noise>
-        <type>gaussian</type>
-        <mean>0.0</mean>
-        <stddev>0.001</stddev>
-      </noise>
-    </ray>
-    <always_on>0</always_on>
-    <update_rate>20</update_rate>
-    <visualize>false</visualize>
-  </sensor>
-</gazebo>
+    <origin rpy="0 0 0" xyz="-0.1 0 0.268"/>
+  </joint>
+  <gazebo reference="lidar_2d_v1">
+    <sensor name="lidar_2d_v1" type="gpu_ray">
+      <topic>lidar</topic>
+      <ignition_frame_id>lidar_2d_v1</ignition_frame_id>
+      <pose>0 0 0.0525045525 0 0 0</pose>
+      <ray>
+        <scan>
+          <horizontal>
+            <samples>90</samples>
+            <resolution>1</resolution>
+            <min_angle>-1.41</min_angle>
+            <max_angle>1.41</max_angle>
+          </horizontal>
+        </scan>
+        <range>
+          <min>0.060</min>
+          <max>10</max>
+          <resolution>0.04</resolution>
+        </range>
+        <noise>
+          <type>gaussian</type>
+          <mean>0.0</mean>
+          <stddev>0.001</stddev>
+        </noise>
+      </ray>
+      <always_on>0</always_on>
+      <update_rate>20</update_rate>
+      <visualize>false</visualize>
+    </sensor>
+  </gazebo>
 </robot>

Commit message: Adding haul_truck example

File: src/start_creating_robots/worlds_and_models/krytn/krytn.urdf.xacro (robot description, xacro)
@@ -1,4 +1,7 @@
 <?xml version='1.0' encoding='utf-8'?>
 <robot xmlns:xacro="http://www.ros.org/wiki/xacro" name="krytn">
+    <material name="blue">
+        <color rgba="0 0 0.8 1"/>
+    </material>
     <xacro:arg name="with_sensors" default="true" />
     <!-- Include the robot base. Configure it with a differential drive control plugin -->
@@ -16,4 +19,5 @@
                     <mesh filename="file://$(find start_creating_robots)/worlds_and_models/krytn/meshes/krytn_top-part.dae"/>
                 </geometry>
+                <material name="blue" />
             </visual>
         </link>
