Commit message: Developing scorpion

File: src/start_creating_robots/worlds_and_models/krytn/realsense_d435.urdf.xacro (robot description, xacro)
@@ -1,6 +1,6 @@
 <?xml version="1.0"?>
 <robot xmlns:xacro="http://wiki.ros.org/xacro">
-<link name="realsense_d435">
-  <origin xyz="0.2 0 0.2" rpy="0 0 0" />
+  <link name="realsense_d435">
+    <origin xyz="0.2 0 0.2" rpy="0 0 0" />
     <collision name="collision">
       <geometry>
@@ -18,59 +18,59 @@
       </geometry>
     </visual>
-</link>
-<joint name="depth_camera_joint" type="fixed">
-        <parent link="base_footprint" />
-        <child link="realsense_d435" />
-        <origin rpy="0 0 0" xyz="0 0 0.6"/>
-</joint>
-<gazebo reference="realsense_d435">
-  <sensor name="realsense_d435" type="rgbd_camera">
-    <topic>realsense</topic>
-    <ignition_frame_id>realsense_d435</ignition_frame_id>
-    <update_rate>5</update_rate>
-    <camera name="camera">
-      <horizontal_fov>0.5</horizontal_fov>
-      <lens>
-        <intrinsics>
-          <!-- fx = fy = width / ( 2 * tan (hfov / 2 ) ) -->
-          <fx>554.25469</fx>
-          <fy>554.25469</fy>
-          <!-- cx = ( width + 1 ) / 2 -->
-          <cx>320.5</cx>
-          <!-- cy = ( height + 1 ) / 2 -->
-          <cy>240.5</cy>
-          <s>0</s>
-        </intrinsics>
-      </lens>
-      <distortion>
-        <k1>0.0</k1>
-        <k2>0.0</k2>
-        <k3>0.0</k3>
-        <p1>0.0</p1>
-        <p2>0.0</p2>
-        <center>0.5 0.5</center>
-      </distortion>
-      <image>
-        <width>160</width>
-        <height>120</height>
-        <format>R8G8B8</format>
-      </image>
-      <clip>
-        <near>0.01</near>
-        <far>10</far>
-      </clip>
-      <depth_camera>
+  </link>
+  <joint name="depth_camera_joint" type="fixed">
+    <parent link="base_footprint" />
+    <child link="realsense_d435" />
+    <origin rpy="0 0 0" xyz="0 0 0.6"/>
+  </joint>
+  <gazebo reference="realsense_d435">
+    <sensor name="realsense_d435" type="rgbd_camera">
+      <topic>realsense</topic>
+      <ignition_frame_id>realsense_d435</ignition_frame_id>
+      <update_rate>5</update_rate>
+      <camera name="camera">
+        <horizontal_fov>0.5</horizontal_fov>
+        <lens>
+          <intrinsics>
+            <!-- fx = fy = width / ( 2 * tan (hfov / 2 ) ) -->
+            <fx>554.25469</fx>
+            <fy>554.25469</fy>
+            <!-- cx = ( width + 1 ) / 2 -->
+            <cx>320.5</cx>
+            <!-- cy = ( height + 1 ) / 2 -->
+            <cy>240.5</cy>
+            <s>0</s>
+          </intrinsics>
+        </lens>
+        <distortion>
+          <k1>0.0</k1>
+          <k2>0.0</k2>
+          <k3>0.0</k3>
+          <p1>0.0</p1>
+          <p2>0.0</p2>
+          <center>0.5 0.5</center>
+        </distortion>
+        <image>
+          <width>160</width>
+          <height>120</height>
+          <format>R8G8B8</format>
+        </image>
         <clip>
-          <near>0.1</near>
+          <near>0.01</near>
           <far>10</far>
         </clip>
-      </depth_camera>
-      <noise>
-        <type>gaussian</type>
-        <mean>0</mean>
-        <stddev>0.007</stddev>
-      </noise>
-    </camera>
-  </sensor>
-</gazebo>
+        <depth_camera>
+          <clip>
+            <near>0.1</near>
+            <far>10</far>
+          </clip>
+        </depth_camera>
+        <noise>
+          <type>gaussian</type>
+          <mean>0</mean>
+          <stddev>0.007</stddev>
+        </noise>
+      </camera>
+    </sensor>
+  </gazebo>
 </robot>

File: src/veg_bot/worlds_and_models/kuka/kr6r900sixx.xacro (robot description, xacro)
@@ -4,4 +4,5 @@
   <xacro:include filename="$(find veg_bot)/worlds_and_models/kuka/kr6r900sixx_macro.xacro" />
   <xacro:kuka_kr6r900sixx prefix=""/>
+  <xacro:include filename="$(find veg_bot)/worlds_and_models/kuka/realsense.urdf.xacro" />
   <gazebo>
     <plugin filename="ignition-gazebo-detachable-joint-system" name="ignition::gazebo::systems::DetachableJoint">
@@ -13,4 +14,7 @@
       <output_topic>/lemon/state</output_topic>
     </plugin>
+    <plugin filename="ignition-gazebo-sensors-system" name="ignition::gazebo::systems::Sensors">
+      <render_engine>ogre2</render_engine>
+    </plugin>
   </gazebo>
 </robot>
