Commit message: Added control

File: src/scorpion/worlds_and_models/scorpion/scorpion.urdf.xacro (robot description, xacro)
@@ -1,6 +1,20 @@
 <?xml version="1.0" ?>
-<robot name="kuka_kr6"
+<robot name="scorpion"
     xmlns:xacro="http://wiki.ros.org/xacro">
+    <material name="red">
+        <color rgba="1 0.0 0.0 1"/>
+    </material>
+    <material name="black">
+        <color rgba="0.043 0.004 0 1"/>
+    </material>
+    <material name="silver">
+        <color rgba="0.73 0.73 0.82 1"/>
+    </material>
     <xacro:include filename="$(find start_creating_robots)/worlds_and_models/krytn/inertial.xacro" />
+    <link name="base_link" />
+    <joint name="chasis_link_joint" type="fixed">
+        <parent link="base_link" />
+        <child link="chassis_link" />
+    </joint>
     <!--Generated by CROSS, a ROS Workbench for FreeCAD (https://github.com/galou/freecad.cross)-->
     <link name="chassis_link">
@@ -11,4 +25,5 @@
                 <mesh filename="file://$(find scorpion)/worlds_and_models/scorpion/meshes/Unnamed_chassis_body.dae"/>
             </geometry>
+            <material name="red" />
         </visual>
         <collision>
@@ -18,5 +33,5 @@
             </geometry>
         </collision>
-        <xacro:box_inertial_with_origin x="0.18" y="0.09" z="0.15" mass="3">
+        <xacro:box_inertial_with_origin x="0.18" y="0.09" z="0.15" mass="4">
             <origin xyz="0.09 0 0" />
         </xacro:box_inertial_with_origin>
@@ -29,4 +44,5 @@
                 <mesh filename="file://$(find scorpion)/worlds_and_models/scorpion/meshes/Unnamed_tail1_body.dae"/>
             </geometry>
+            <material name="red" />
         </visual>
         <collision>
@@ -47,4 +63,5 @@
                 <mesh filename="file://$(find scorpion)/worlds_and_models/scorpion/meshes/Unnamed_tail2_body.dae"/>
             </geometry>
+            <material name="black" />
         </visual>
         <collision>
@@ -54,5 +71,5 @@
             </geometry>
         </collision>
-        <xacro:box_inertial_with_origin x="0.05" y="0.03" z="0.045" mass="0.4">
+        <xacro:box_inertial_with_origin x="0.05" y="0.03" z="0.045" mass="0.2">
             <origin xyz="-0.025 0 0" />
         </xacro:box_inertial_with_origin>
@@ -65,10 +82,11 @@
                 <mesh filename="file://$(find scorpion)/worlds_and_models/scorpion/meshes/Unnamed_tail3_body.dae"/>
             </geometry>
-        </visual>
-        <xacro:box_inertial_with_origin x="0.1" y="0.025" z="0.054" mass="0.8">
+            <material name="silver" />
+        </visual>
+        <xacro:box_inertial_with_origin x="0.1" y="0.025" z="0.054" mass="0.4">
             <origin xyz="-0.05 0 0" />
         </xacro:box_inertial_with_origin>
         <collision>
-            <origin xyz="-0.05 0 0" />
+            <origin xyz="-0.05 0 0" rpy="1.57 0 0" />
             <geometry>
                 <box size="0.1 0.025 0.054" />
@@ -84,9 +102,10 @@
                     <mesh filename="file://$(find scorpion)/worlds_and_models/scorpion/meshes/Unnamed_wheel_body.dae"/>
                 </geometry>
+                <material name="black" />
             </visual>
             <collision>
                 <origin rpy="1.57 0 0" />
                 <geometry>
-                    <cylinder radius="0.02" length="0.005" />
+                    <cylinder radius="0.02" length="0.02" />
                 </geometry>
             </collision>
@@ -109,6 +128,6 @@
         <child link="tail_link1"/>
         <origin xyz="0.19 0.0 0.05" rpy="0.0 0.7853981633974484 0.0"/>
-        <axis xyz="0 1 0"/>
-        <limit lower="0.0" upper="3.141592653589793" velocity="10" effort="10.0"/>
+        <axis xyz="0 -1 0"/>
+        <limit upper="3.14" lower="-3.141592653589793" velocity="10" effort="10.0"/>
     </joint>
     <joint name="joint_2" type="revolute">
@@ -123,5 +142,5 @@
         <child link="tail_link3"/>
         <origin xyz="-0.046 0.0 0.0" rpy="0.0 -0.0 0.0"/>
-        <axis xyz="0 1 0"/>
+        <axis xyz="0 -1 0"/>
         <limit lower="-1.5707963267948966" upper="1.5707963267948966" velocity="1" effort="10.0"/>
     </joint>
@@ -131,5 +150,5 @@
             <child link="${side}_wheel_${num}"/>
             <origin xyz="${xyz}" rpy="0 0 0"/>
-            <axis xyz="0 1 0"/>
+            <axis xyz="0 -1 0"/>
             <limit lower="-10000.0" upper="10000.0" velocity="1" effort="10.0"/>
         </joint>
@@ -141,3 +160,51 @@
     <xacro:make_wheel_joint xyz="0.09 0.033 0.015" side="right" num="2" />
     <xacro:make_wheel_joint xyz="0.16 0.033 0.015" side="right" num="3" />
+    <xacro:macro name="ros2_control_wheel_joint" params="side num">
+        <joint name="${side}_wheel_joint_${num}">
+            <command_interface name="velocity">
+                <param name="min">-0.2</param>
+                <param name="max">0.2</param>
+            </command_interface>
+            <state_interface name="position"/>
+            <state_interface name="velocity"/>
+        </joint>
+    </xacro:macro>
+    <xacro:macro name="ros2_control_make_side_wheels" params="side num">
+        <xacro:if value="${num > 0}">
+            <xacro:ros2_control_wheel_joint side="${side}" num="${num}" />
+            <xacro:ros2_control_make_side_wheels side="${side}" num="${num-1}" />
+        </xacro:if>
+    </xacro:macro>
+    <xacro:macro name="ros2_control_tail_joint" params="num minj maxj">
+        <joint name="joint_${num}">
+            <command_interface name="position">
+                <param name="min">${minj}</param>
+                <param name="max">${maxj}</param>
+            </command_interface>
+            <state_interface name="position"/>
+            <state_interface name="velocity"/>
+        </joint>
+    </xacro:macro>
+    <ros2_control name="GazeboSystem" type="system">
+        <hardware>
+            <plugin>ign_ros2_control/IgnitionSystem</plugin>
+        </hardware>
+        <!-- Using Xacro to minimise boilerplate code -->
+        <xacro:ros2_control_make_side_wheels side="left" num="3" />
+        <xacro:ros2_control_make_side_wheels side="right" num="3" />
+        <xacro:ros2_control_tail_joint num="1" minj="0" maxj="3.14" />
+        <xacro:ros2_control_tail_joint num="2" minj="-1.57" maxj="1.57" />
+        <xacro:ros2_control_tail_joint num="3" minj="-1.57" maxj="1.57" />
+    </ros2_control>
+    <gazebo>
+        <plugin filename="ign_ros2_control-system" name="ign_ros2_control::IgnitionROS2ControlPlugin">
+            <ros>
+                <remapping>/diff_drive_base_controller/odometry:=odom</remapping>
+                <remapping>/diff_drive_base_controller/tf_odometry:=tf</remapping>
+                <remapping>/diff_drive_base_controller/cmd_vel_unstamped:=cmd_vel</remapping>
+            </ros>
+            <parameters>$(find scorpion)/config/diffdrive_control.yaml</parameters>
+        </plugin>
+        <!-- Remapping topics so that mapping system works! -->
+    </gazebo>
 </robot>

Commit message: Got scorpion working ok

File: src/scorpion/worlds_and_models/scorpion/scorpion.urdf.xacro (robot description, xacro)
@@ -16,4 +16,5 @@
         <parent link="base_link" />
         <child link="chassis_link" />
+        <origin xyz="0 0 0" rpy="0 0 3.141" />
     </joint>
     <!--Generated by CROSS, a ROS Workbench for FreeCAD (https://github.com/galou/freecad.cross)-->
@@ -114,4 +115,18 @@
             </xacro:cylinder_inertial_with_origin>
         </link>
+        <gazebo reference="${side}_wheel_${num}">
+            <collision>
+                <surface>
+                    <friction>
+                        <ode>
+                            <mu>0.5</mu>
+                            <mu1>0.5</mu1>
+                            <mu2>1.0</mu2>
+                            <fdir1>0 0 1</fdir1>
+                        </ode>
+                    </friction>
+                </surface>
+            </collision>
+        </gazebo>
     </xacro:macro>
     <!-- Example of a tail-recursion loop in Xacro. This macro calls itself with 1 minus its given value. -->
@@ -200,5 +215,5 @@
         <plugin filename="ign_ros2_control-system" name="ign_ros2_control::IgnitionROS2ControlPlugin">
             <ros>
-                <remapping>/diff_drive_base_controller/odometry:=odom</remapping>
+                <remapping>/diff_drive_base_controller/odom:=odom</remapping>
                 <remapping>/diff_drive_base_controller/tf_odometry:=tf</remapping>
                 <remapping>/diff_drive_base_controller/cmd_vel_unstamped:=cmd_vel</remapping>
@@ -207,45 +222,34 @@
         </plugin>
         <!-- Remapping topics so that mapping system works! -->
+        <plugin filename="ignition-gazebo-sensors-system" name="ignition::gazebo::systems::Sensors">
+            <render_engine>ogre2</render_engine>
+        </plugin>
     </gazebo>
-    <gazebo reference="chassis_link">
+    <link name="chassis_camera_link" />
+    <joint name="chassis_camera_joint" type="fixed">
+        <parent link="chassis_link"/>
+        <child link="chassis_camera_link" />
+        <origin xyz="0 0 0.1" rpy="0 0 3.141" />
+    </joint>
+    <gazebo reference="chassis_camera_link">
         <sensor name="realsense_d435" type="rgbd_camera">
             <topic>realsense</topic>
-            <ignition_frame_id>chassis_link</ignition_frame_id>
+            <ignition_frame_id>chassis_camera_optical_link</ignition_frame_id>
             <update_rate>5</update_rate>
             <camera name="depth_camera">
-                <horizontal_fov>0.5</horizontal_fov>
-                <lens>
-                    <intrinsics>
-                        <!-- fx = fy = width / ( 2 * tan (hfov / 2 ) ) -->
-                        <fx>554.25469</fx>
-                        <fy>554.25469</fy>
-                        <!-- cx = ( width + 1 ) / 2 -->
-                        <cx>320.5</cx>
-                        <!-- cy = ( height + 1 ) / 2 -->
-                        <cy>240.5</cy>
-                        <s>0</s>
-                    </intrinsics>
-                </lens>
-                <distortion>
-                    <k1>0.0</k1>
-                    <k2>0.0</k2>
-                    <k3>0.0</k3>
-                    <p1>0.0</p1>
-                    <p2>0.0</p2>
-                    <center>0.5 0.5</center>
-                </distortion>
+                <horizontal_fov>1.4</horizontal_fov>
                 <image>
-                    <width>160</width>
-                    <height>120</height>
+                    <width>640</width>
+                    <height>480</height>
                     <format>R8G8B8</format>
                 </image>
                 <clip>
                     <near>0.01</near>
-                    <far>10</far>
+                    <far>5</far>
                 </clip>
                 <depth_camera>
                     <clip>
                         <near>0.1</near>
-                        <far>10</far>
+                        <far>5</far>
                     </clip>
                 </depth_camera>
@@ -258,41 +262,29 @@
         </sensor>
     </gazebo>
-    <gazebo reference="tail_link3">
-        <sensor name="realsense_d435" type="camera">
+    <link name="tail_camera_link"/>
+    <joint name="tail_camera_joint" type="fixed">
+        <parent link="tail_link3" />
+        <child link="tail_camera_link" />
+        <origin xyz="-0.25 0 0" rpy="0 0 3.141"/>
+    </joint>
+    <gazebo reference="tail_camera_link">
+        <sensor name="tailcamera" type="camera">
             <topic>tail_camera</topic>
-            <ignition_frame_id>tail_link3</ignition_frame_id>
+            <ignition_frame_id>tail_camera_link</ignition_frame_id>
             <update_rate>5</update_rate>
-            <camera name="tail_cam">
-                <horizontal_fov>0.5</horizontal_fov>
-                <lens>
-                    <intrinsics>
-                        <!-- fx = fy = width / ( 2 * tan (hfov / 2 ) ) -->
-                        <fx>554.25469</fx>
-                        <fy>554.25469</fy>
-                        <!-- cx = ( width + 1 ) / 2 -->
-                        <cx>320.5</cx>
-                        <!-- cy = ( height + 1 ) / 2 -->
-                        <cy>240.5</cy>
-                        <s>0</s>
-                    </intrinsics>
-                </lens>
-                <distortion>
-                    <k1>0.0</k1>
-                    <k2>0.0</k2>
-                    <k3>0.0</k3>
-                    <p1>0.0</p1>
-                    <p2>0.0</p2>
-                    <center>0.5 0.5</center>
-                </distortion>
+            <camera>
+                <horizontal_fov>1.047</horizontal_fov>
                 <image>
-                    <width>160</width>
-                    <height>120</height>
-                    <format>R8G8B8</format>
+                    <width>320</width>
+                    <height>240</height>
                 </image>
                 <clip>
-                    <near>0.01</near>
-                    <far>10</far>
+                    <near>0.1</near>
+                    <far>20</far>
                 </clip>
             </camera>
+            <always_on>1</always_on>
+            <update_rate>5</update_rate>
+            <visualize>true</visualize>
         </sensor>
     </gazebo>
