Commit message: ros2 diff drive working!

File: src/haul_truck/worlds_and_models/haul_truck/Haul_Truck.urdf.xacro (robot description, xacro)
@@ -11,4 +11,9 @@
   </material>
   <xacro:include filename="$(find start_creating_robots)/worlds_and_models/krytn/inertial.xacro" />
+  <link name="base_link" />
+  <joint name="chassis_joint" type="fixed">
+    <parent link="base_link" />
+    <child link="chassis_link" />
+  </joint>
   <!--Generated by CROSS, a ROS Workbench for FreeCAD (https://github.com/galou/freecad.cross)-->
   <link name="chassis_link">
@@ -156,5 +161,4 @@
     <origin xyz="2.8 3.2 0.0" rpy="0.0 -0.0 0.0"/>
     <axis xyz="1 0 0"/>
-    <limit lower="0.0" upper="0.0" velocity="0.0" effort="0.0"/>
   </joint>
   <joint name="front_right_wheel_joint" type="continuous">
@@ -163,5 +167,4 @@
     <origin xyz="-4.0 3.2 0.0" rpy="0.0 -0.0 0.0"/>
     <axis xyz="1 0 0"/>
-    <limit lower="0.0" upper="0.0" velocity="0.0" effort="0.0"/>
   </joint>
   <joint name="rear_left_wheel_joint" type="continuous">
@@ -170,5 +173,4 @@
     <origin xyz="2.8 9.3 0.0" rpy="0.0 -0.0 0.0"/>
     <axis xyz="1 0 0"/>
-    <limit lower="0.0" upper="0.0" velocity="0.0" effort="0.0"/>
   </joint>
   <joint name="rear_right_wheel_joint" type="continuous">
@@ -177,5 +179,4 @@
     <origin xyz="-4.0 9.3 0.0" rpy="0.0 -0.0 0.0"/>
     <axis xyz="1 0 0"/>
-    <limit lower="0.0" upper="0.0" velocity="0.0" effort="0.0"/>
   </joint>
   <xacro:include filename="$(find haul_truck)/worlds_and_models/haul_truck/lidar_3d_v1.urdf.xacro" />
@@ -185,3 +186,46 @@
     </plugin>
   </gazebo>
+  <ros2_control name="GazeboSystem" type="system">
+    <hardware>
+      <plugin>ign_ros2_control/IgnitionSystem</plugin>
+    </hardware>
+    <joint name="front_left_wheel_joint">
+      <command_interface name="velocity">
+        <param name="min">-1</param>
+        <param name="max">1</param>
+      </command_interface>
+      <state_interface name="position"/>
+      <state_interface name="velocity"/>
+    </joint>
+    <joint name="front_right_wheel_joint">
+      <command_interface name="velocity">
+        <param name="min">-1</param>
+        <param name="max">1</param>
+      </command_interface>
+      <state_interface name="position"/>
+      <state_interface name="velocity"/>
+    </joint>
+    <joint name="rear_left_wheel_joint">
+      <command_interface name="velocity">
+        <param name="min">-1</param>
+        <param name="max">1</param>
+      </command_interface>
+      <state_interface name="position"/>
+      <state_interface name="velocity"/>
+    </joint>
+    <joint name="rear_right_wheel_joint">
+      <command_interface name="velocity">
+        <param name="min">-1</param>
+        <param name="max">1</param>
+      </command_interface>
+      <state_interface name="position"/>
+      <state_interface name="velocity"/>
+    </joint>
+  </ros2_control>
+  <gazebo>
+    <!-- Joint state publisher -->
+    <plugin filename="ign_ros2_control-system" name="ign_ros2_control::IgnitionROS2ControlPlugin">
+      <parameters>$(find haul_truck)/config/diffdrive_control.yaml</parameters>
+    </plugin>
+  </gazebo>
 </robot>

Commit message: developing ackermann steering

File: src/haul_truck/worlds_and_models/haul_truck/Haul_Truck.urdf.xacro (robot description, xacro)
@@ -151,4 +151,24 @@
     <xacro:sphere_inertial radius="1" mass="2000" />
   </link>
+  <link name="front_left_steering_link">
+    <xacro:box_inertial x="0.1" y="1" z="0.1" mass="1"/>
+  </link>
+  <link name="front_right_steering_link">
+    <xacro:box_inertial x="0.1" y="1" z="0.1" mass="1"/>
+  </link>
+  <joint name="front_left_steering_joint" type="revolute">
+    <parent link="chassis_link" />
+    <child link="front_left_steering_link" />
+    <axis xyz="0 0 1"/>
+    <origin xyz="2.8 3.2 0.0" rpy="0.0 -0.0 0.0"/>
+    <limit lower="-0.8727" upper="0.8727" effort="1000" velocity="1000.00"/>
+  </joint>
+  <joint name="front_right_steering_joint" type="revolute">
+    <parent link="chassis_link" />
+    <child link="front_right_steering_link" />
+    <origin xyz="-2.8 3.2 0.0" rpy="0.0 -0.0 0.0"/>
+    <axis xyz="0 0 1"/>
+    <limit lower="-0.8727" upper="0.8727" effort="1000" velocity="1000.00"/>
+  </joint>
   <joint name="tray_joint" type="fixed">
     <parent link="chassis_link"/>
@@ -157,13 +177,11 @@
   </joint>
   <joint name="front_left_wheel_joint" type="continuous">
-    <parent link="chassis_link"/>
+    <parent link="front_left_steering_link"/>
     <child link="front_left_wheel_link"/>
-    <origin xyz="2.8 3.2 0.0" rpy="0.0 -0.0 0.0"/>
     <axis xyz="1 0 0"/>
   </joint>
   <joint name="front_right_wheel_joint" type="continuous">
-    <parent link="chassis_link"/>
+    <parent link="front_right_steering_link"/>
     <child link="front_right_wheel_link"/>
-    <origin xyz="-4.0 3.2 0.0" rpy="0.0 -0.0 0.0"/>
     <axis xyz="1 0 0"/>
   </joint>
@@ -171,5 +189,5 @@
     <parent link="chassis_link"/>
     <child link="rear_left_wheel_link"/>
-    <origin xyz="2.8 9.3 0.0" rpy="0.0 -0.0 0.0"/>
+    <origin xyz="4.0 9.3 0.0" rpy="0.0 -0.0 0.0"/>
     <axis xyz="1 0 0"/>
   </joint>
@@ -190,4 +208,18 @@
       <plugin>ign_ros2_control/IgnitionSystem</plugin>
     </hardware>
+    <joint name="front_left_steering_wheel_joint">
+      <command_interface name="position">
+        <param name="min">-0.8727</param>
+        <param name="max">0.8727</param>
+      </command_interface>
+      <state_interface name="position"/>
+    </joint>
+    <joint name="front_right_steering_wheel_joint">
+      <command_interface name="position">
+        <param name="min">-0.8727</param>
+        <param name="max">0.8727</param>
+      </command_interface>
+      <state_interface name="position"/>
+    </joint>
     <joint name="front_left_wheel_joint">
       <command_interface name="velocity">
@@ -224,5 +256,4 @@
   </ros2_control>
   <gazebo>
-    <!-- Joint state publisher -->
     <plugin filename="ign_ros2_control-system" name="ign_ros2_control::IgnitionROS2ControlPlugin">
       <parameters>$(find haul_truck)/config/diffdrive_control.yaml</parameters>

Commit message: Added simulation world

File: src/haul_truck/worlds_and_models/haul_truck/Haul_Truck.urdf.xacro (robot description, xacro)
@@ -22,7 +22,6 @@
       <origin xyz="0.0 0.0 0.0" rpy="0.0 -0.0 0.0"/>
       <geometry>
-        <mesh filename="package://haul_truck/meshes/Unnamed_Body.dae"/>
-      </geometry>
-      <material name="orange" />
+        <mesh filename="package://haul_truck/meshes/safeai_Body.dae"/>
+      </geometry>
     </visual>
     <collision>
@@ -36,5 +35,5 @@
       </gazebo>
     </collision>
-    <xacro:box_inertial_with_origin x="8" y="10" z="3" mass="100000">
+    <xacro:box_inertial_with_origin x="8" y="10" z="3" mass="100">
       <origin xyz="0 5 0" rpy="0 0 0" />
     </xacro:box_inertial_with_origin>
@@ -49,9 +48,9 @@
       <material name="red" />
     </visual>
-    <collision>
-      <!--real_tray_link_.Body002_bbox-->
-      <origin xyz="0.219 7.17182 5.93052" rpy="0.0 -0.0 0.0"/>
-      <geometry>
-        <box size="7.638000000000004 13.858283829000012 3.4610417480000075"/>
+    <!--
+    <collision>
+      <origin xyz="3.5 7 0 " rpy="0.0 -0.0 0.0"/>
+      <geometry>
+        <box size="7.638000000000004 13.858283829000012 1.4610417480000075"/>
       </geometry>
       <gazebo>
@@ -59,7 +58,8 @@
       </gazebo>
     </collision>
-    <xacro:box_inertial_with_origin x="8" y="10" z="1" mass="10000">
+    <xacro:box_inertial_with_origin x="8" y="10" z="1" mass="1">
       <origin xyz="0 -5 0" rpy="0 0 0" />
     </xacro:box_inertial_with_origin>
+  -->
   </link>
   <link name="front_left_wheel_link">
@@ -68,18 +68,20 @@
       <origin xyz="0.0 0.0 0.0" rpy="0.0 -0.0 0.0"/>
       <geometry>
-        <mesh filename="package://haul_truck/meshes/Unnamed_Body001.dae"/>
-      </geometry>
-      <material name="black" />
-    </visual>
-    <collision>
-      <!--Wheel/Body001.-->
-      <origin xyz="0.0 0.0 0.0" rpy="0.0 -0.0 0.0"/>
-      <geometry>
-        <mesh filename="package://haul_truck/meshes/Unnamed_Body001.dae"/>
-      </geometry>
-    </collision>
-    <xacro:sphere_inertial radius="1" mass="2000" />
+        <mesh filename="package://haul_truck/meshes/safeai_Body001.dae"/>
+      </geometry>
+      <material name="black" />
+    </visual>
+    <collision>
+      <!--Wheel/Body001.-->
+      <origin xyz="0.0 0.0 0.0" rpy="0.0 -0.0 0.0"/>
+      <geometry>
+        <mesh filename="package://haul_truck/meshes/safeai_Pad012.dae"/>
+      </geometry>
+    </collision>
+    <xacro:cylinder_inertial_with_origin radius="1" length="0.5" mass="2">
+      <origin rpy="0 0 0.57"/>
+    </xacro:cylinder_inertial_with_origin>
     <gazebo>
-      <mu>0.3</mu>
+      <mu>0.7</mu>
       <minDepth>0.02</minDepth>
     </gazebo>
@@ -90,20 +92,22 @@
       <origin xyz="0.0 0.0 0.0" rpy="0.0 -0.0 0.0"/>
       <geometry>
-        <mesh filename="package://haul_truck/meshes/Unnamed_Body001.dae"/>
-      </geometry>
-      <material name="black" />
-    </visual>
-    <collision>
-      <!--Wheel/Body001.-->
-      <origin xyz="0.0 0.0 0.0" rpy="0.0 -0.0 0.0"/>
-      <geometry>
-        <mesh filename="package://haul_truck/meshes/Unnamed_Body001.dae"/>
-      </geometry>
-      <gazebo>
-        <mu>0.3</mu>
+        <mesh filename="package://haul_truck/meshes/safeai_Body001.dae"/>
+      </geometry>
+      <material name="black" />
+    </visual>
+    <collision>
+      <!--Wheel/Body001.-->
+      <origin xyz="0.0 0.0 0.0" rpy="0.0 -0.0 0.0"/>
+      <geometry>
+        <mesh filename="package://haul_truck/meshes/safeai_Pad012.dae"/>
+      </geometry>
+      <gazebo>
+        <mu>0.7</mu>
         <minDepth>0.02</minDepth>
       </gazebo>
     </collision>
-    <xacro:sphere_inertial radius="1" mass="2000" />
+    <xacro:cylinder_inertial_with_origin radius="1" length="0.5" mass="2">
+      <origin rpy="0 0 0.57"/>
+    </xacro:cylinder_inertial_with_origin>
   </link>
   <link name="rear_left_wheel_link">
@@ -112,20 +116,20 @@
       <origin xyz="0.0 0.0 0.0" rpy="0.0 -0.0 0.0"/>
       <geometry>
-        <mesh filename="package://haul_truck/meshes/Unnamed_Body001.dae"/>
-      </geometry>
-      <material name="black" />
-    </visual>
-    <collision>
-      <!--Wheel/Body001.-->
-      <origin xyz="0.0 0.0 0.0" rpy="0.0 -0.0 0.0"/>
-      <geometry>
-        <mesh filename="package://haul_truck/meshes/Unnamed_Body001.dae"/>
-      </geometry>
-      <gazebo>
-        <mu>0.3</mu>
+        <mesh filename="package://haul_truck/meshes/safeai_Body001.dae"/>
+      </geometry>
+      <material name="black" />
+    </visual>
+    <collision>
+      <!--Wheel/Body001.-->
+      <origin xyz="0.0 0.0 0.0" rpy="0.0 -0.0 0.0"/>
+      <geometry>
+        <mesh filename="package://haul_truck/meshes/safeai_Pad012.dae"/>
+      </geometry>
+      <gazebo>
+        <mu>0.7</mu>
         <minDepth>0.02</minDepth>
       </gazebo>
     </collision>
-    <xacro:sphere_inertial radius="1" mass="2000" />
+    <xacro:sphere_inertial radius="1" mass="2" />
   </link>
   <link name="rear_right_wheel_link">
@@ -134,20 +138,20 @@
       <origin xyz="0.0 0.0 0.0" rpy="0.0 -0.0 0.0"/>
       <geometry>
-        <mesh filename="package://haul_truck/meshes/Unnamed_Body001.dae"/>
-      </geometry>
-      <material name="black" />
-    </visual>
-    <collision>
-      <!--Wheel/Body001.-->
-      <origin xyz="0.0 0.0 0.0" rpy="0.0 -0.0 0.0"/>
-      <geometry>
-        <mesh filename="package://haul_truck/meshes/Unnamed_Body001.dae"/>
-      </geometry>
-      <gazebo>
-        <mu>0.3</mu>
+        <mesh filename="package://haul_truck/meshes/safeai_Body001.dae"/>
+      </geometry>
+      <material name="black" />
+    </visual>
+    <collision>
+      <!--Wheel/Body001.-->
+      <origin xyz="0.0 0.0 0.0" rpy="0.0 -0.0 0.0"/>
+      <geometry>
+        <mesh filename="package://haul_truck/meshes/safeai_Pad012.dae"/>
+      </geometry>
+      <gazebo>
+        <mu>0.7</mu>
         <minDepth>0.02</minDepth>
       </gazebo>
     </collision>
-    <xacro:sphere_inertial radius="1" mass="2000" />
+    <xacro:sphere_inertial radius="1" mass="2" />
   </link>
   <link name="front_left_steering_link">
@@ -161,18 +165,18 @@
     <child link="front_left_steering_link" />
     <axis xyz="0 0 1"/>
-    <origin xyz="2.8 3.2 0.0" rpy="0.0 -0.0 0.0"/>
-    <limit lower="-0.8727" upper="0.8727" effort="1000" velocity="1000.00"/>
+    <origin xyz="2.8 3.2 0.6" rpy="0.0 -0.0 0.0"/>
+    <limit lower="-0.4" upper="0.4" effort="10000000" velocity="1000.00"/>
   </joint>
   <joint name="front_right_steering_joint" type="revolute">
     <parent link="chassis_link" />
     <child link="front_right_steering_link" />
-    <origin xyz="-2.8 3.2 0.0" rpy="0.0 -0.0 0.0"/>
+    <origin xyz="-4.0 3.2 0.6" rpy="0.0 -0.0 0.0"/>
     <axis xyz="0 0 1"/>
-    <limit lower="-0.8727" upper="0.8727" effort="1000" velocity="1000.00"/>
+    <limit lower="-0.4" upper="0.4" effort="10000000" velocity="1000.00"/>
   </joint>
   <joint name="tray_joint" type="fixed">
     <parent link="chassis_link"/>
     <child link="tray_link"/>
-    <origin xyz="-3.6 0.1 4.2" rpy="0.0 -0.0 0.0"/>
+    <origin xyz="-3.8 1.0 3.1" rpy="0.0 -0.0 0.0"/>
   </joint>
   <joint name="front_left_wheel_joint" type="continuous">
@@ -189,5 +193,5 @@
     <parent link="chassis_link"/>
     <child link="rear_left_wheel_link"/>
-    <origin xyz="4.0 9.3 0.0" rpy="0.0 -0.0 0.0"/>
+    <origin xyz="2.8 9.3 0.6" rpy="0.0 -0.0 0.0"/>
     <axis xyz="1 0 0"/>
   </joint>
@@ -195,5 +199,5 @@
     <parent link="chassis_link"/>
     <child link="rear_right_wheel_link"/>
-    <origin xyz="-4.0 9.3 0.0" rpy="0.0 -0.0 0.0"/>
+    <origin xyz="-4.0 9.3 0.6" rpy="0.0 -0.0 0.0"/>
     <axis xyz="1 0 0"/>
   </joint>
@@ -208,5 +212,5 @@
       <plugin>ign_ros2_control/IgnitionSystem</plugin>
     </hardware>
-    <joint name="front_left_steering_wheel_joint">
+    <joint name="front_left_steering_joint">
       <command_interface name="position">
         <param name="min">-0.8727</param>
@@ -215,5 +219,5 @@
       <state_interface name="position"/>
     </joint>
-    <joint name="front_right_steering_wheel_joint">
+    <joint name="front_right_steering_joint">
       <command_interface name="position">
         <param name="min">-0.8727</param>
@@ -221,20 +225,4 @@
       </command_interface>
       <state_interface name="position"/>
-    </joint>
-    <joint name="front_left_wheel_joint">
-      <command_interface name="velocity">
-        <param name="min">-1</param>
-        <param name="max">1</param>
-      </command_interface>
-      <state_interface name="position"/>
-      <state_interface name="velocity"/>
-    </joint>
-    <joint name="front_right_wheel_joint">
-      <command_interface name="velocity">
-        <param name="min">-1</param>
-        <param name="max">1</param>
-      </command_interface>
-      <state_interface name="position"/>
-      <state_interface name="velocity"/>
     </joint>
     <joint name="rear_left_wheel_joint">
@@ -257,5 +245,5 @@
   <gazebo>
     <plugin filename="ign_ros2_control-system" name="ign_ros2_control::IgnitionROS2ControlPlugin">
-      <parameters>$(find haul_truck)/config/diffdrive_control.yaml</parameters>
+      <parameters>$(find haul_truck)/config/ackermann_control.yaml</parameters>
     </plugin>
   </gazebo>

File: src/haul_truck/worlds_and_models/haul_truck/lidar_3d_v1.urdf.xacro (robot description, xacro)
@@ -19,5 +19,6 @@
     <parent link="chassis_link" />
     <child link="lidar_3d_v1" />
-    <origin rpy="0 0 0" xyz="-1 0 6"/>
+    <!--    <origin rpy="0 0 0" xyz="-1 0 6"/> -->
+    <origin xyz="0.0 0.8 5.7" rpy="0.0 -0.0 -1.57"/>
   </joint>
   <gazebo reference="lidar_3d_v1">
@@ -29,20 +30,20 @@
         <scan>
           <horizontal>
-            <samples>90</samples>
-            <resolution>1</resolution>
-            <min_angle>-1.41</min_angle>
-            <max_angle>1.41</max_angle>
-          </horizontal>
-          <vertical>
-            <samples>12</samples>
+            <samples>45</samples>
             <resolution>1</resolution>
             <min_angle>-0.7</min_angle>
             <max_angle>0.7</max_angle>
+          </horizontal>
+          <vertical>
+            <samples>6</samples>
+            <resolution>1</resolution>
+            <min_angle>-0.52</min_angle>
+            <max_angle>0</max_angle>
           </vertical>
         </scan>
         <range>
           <min>0.060</min>
-          <max>10</max>
-          <resolution>0.04</resolution>
+          <max>30</max>
+          <resolution>0.1</resolution>
         </range>
         <noise>
@@ -53,6 +54,6 @@
       </ray>
       <always_on>0</always_on>
-      <update_rate>20</update_rate>
-      <visualize>false</visualize>
+      <update_rate>10</update_rate>
+      <visualize>true</visualize>
     </sensor>
   </gazebo>
