Commit message: Problems with ROS2_control odom preventing a slam solution

File: src/haul_truck/worlds_and_models/haul_truck/Haul_Truck.urdf.xacro (robot description, xacro)
@@ -11,7 +11,34 @@
   </material>
   <xacro:include filename="$(find start_creating_robots)/worlds_and_models/krytn/inertial.xacro" />
-  <link name="base_link" />
+  <xacro:macro name="wheel" params="name">
+    <link name="${name}">
+      <visual>
+        <!--Wheel/Body001.-->
+        <origin xyz="0.0 0.0 0.0" rpy="0.0 -0.0 0.0"/>
+        <geometry>
+          <mesh filename="file://$(find haul_truck)/worlds_and_models/haul_truck/meshes/safeai_Body001.dae"/>
+        </geometry>
+        <material name="black" />
+      </visual>
+      <collision>
+        <!--Wheel/Body001.-->
+        <origin xyz="0.0 0.0 0.0" rpy="0.0 -0.0 0.0"/>
+        <geometry>
+          <mesh filename="file://$(find haul_truck)/worlds_and_models/haul_truck/meshes/safeai_Pad012.dae"/>
+        </geometry>
+        <mu>1.0</mu>
+        <mu2>1.0</mu2>
+        <fdir1>0 0 1</fdir1>
+        <slip1>1.0</slip1>
+        <slip2>1.0</slip2>
+        <min_depth>0.5</min_depth>
+        <kp>1e8</kp>
+      </collision>
+      <xacro:sphere_inertial radius="1" mass="0.2" />
+    </link>
+  </xacro:macro>
+  <link name="base_footprint" />
   <joint name="chassis_joint" type="fixed">
-    <parent link="base_link" />
+    <parent link="base_footprint" />
     <child link="chassis_link" />
   </joint>
@@ -22,5 +49,5 @@
       <origin xyz="0.0 0.0 0.0" rpy="0.0 -0.0 0.0"/>
       <geometry>
-        <mesh filename="package://haul_truck/meshes/safeai_Body.dae"/>
+        <mesh filename="file://$(find haul_truck)/worlds_and_models/haul_truck/meshes/safeai_Body.dae"/>
       </geometry>
     </visual>
@@ -35,5 +62,5 @@
       </gazebo>
     </collision>
-    <xacro:box_inertial_with_origin x="8" y="10" z="3" mass="100">
+    <xacro:box_inertial_with_origin x="8" y="10" z="3" mass="1">
       <origin xyz="0 5 0" rpy="0 0 0" />
     </xacro:box_inertial_with_origin>
@@ -44,5 +71,5 @@
       <origin xyz="0.0 0.0 0.0" rpy="0.0 -0.0 0.0"/>
       <geometry>
-        <mesh filename="package://haul_truck/meshes/Unnamed_Body002.dae"/>
+        <mesh filename="file://$(find haul_truck)/worlds_and_models/haul_truck/meshes/Unnamed_Body002.dae"/>
       </geometry>
       <material name="red" />
@@ -63,116 +90,8 @@
   -->
   </link>
-  <link name="front_left_wheel_link">
-    <visual>
-      <!--Wheel/Body001.-->
-      <origin xyz="0.0 0.0 0.0" rpy="0.0 -0.0 0.0"/>
-      <geometry>
-        <mesh filename="package://haul_truck/meshes/safeai_Body001.dae"/>
-      </geometry>
-      <material name="black" />
-    </visual>
-    <collision>
-      <!--Wheel/Body001.-->
-      <origin xyz="0.0 0.0 0.0" rpy="0.0 -0.0 0.0"/>
-      <geometry>
-        <mesh filename="package://haul_truck/meshes/safeai_Pad012.dae"/>
-      </geometry>
-    </collision>
-    <xacro:cylinder_inertial_with_origin radius="1" length="0.5" mass="2">
-      <origin rpy="0 0 0.57"/>
-    </xacro:cylinder_inertial_with_origin>
-    <gazebo>
-      <mu>0.7</mu>
-      <minDepth>0.02</minDepth>
-    </gazebo>
-  </link>
-  <link name="front_right_wheel_link">
-    <visual>
-      <!--Wheel/Body001.-->
-      <origin xyz="0.0 0.0 0.0" rpy="0.0 -0.0 0.0"/>
-      <geometry>
-        <mesh filename="package://haul_truck/meshes/safeai_Body001.dae"/>
-      </geometry>
-      <material name="black" />
-    </visual>
-    <collision>
-      <!--Wheel/Body001.-->
-      <origin xyz="0.0 0.0 0.0" rpy="0.0 -0.0 0.0"/>
-      <geometry>
-        <mesh filename="package://haul_truck/meshes/safeai_Pad012.dae"/>
-      </geometry>
-      <gazebo>
-        <mu>0.7</mu>
-        <minDepth>0.02</minDepth>
-      </gazebo>
-    </collision>
-    <xacro:cylinder_inertial_with_origin radius="1" length="0.5" mass="2">
-      <origin rpy="0 0 0.57"/>
-    </xacro:cylinder_inertial_with_origin>
-  </link>
-  <link name="rear_left_wheel_link">
-    <visual>
-      <!--Wheel/Body001.-->
-      <origin xyz="0.0 0.0 0.0" rpy="0.0 -0.0 0.0"/>
-      <geometry>
-        <mesh filename="package://haul_truck/meshes/safeai_Body001.dae"/>
-      </geometry>
-      <material name="black" />
-    </visual>
-    <collision>
-      <!--Wheel/Body001.-->
-      <origin xyz="0.0 0.0 0.0" rpy="0.0 -0.0 0.0"/>
-      <geometry>
-        <mesh filename="package://haul_truck/meshes/safeai_Pad012.dae"/>
-      </geometry>
-      <gazebo>
-        <mu>0.7</mu>
-        <minDepth>0.02</minDepth>
-      </gazebo>
-    </collision>
-    <xacro:sphere_inertial radius="1" mass="2" />
-  </link>
-  <link name="rear_right_wheel_link">
-    <visual>
-      <!--Wheel/Body001.-->
-      <origin xyz="0.0 0.0 0.0" rpy="0.0 -0.0 0.0"/>
-      <geometry>
-        <mesh filename="package://haul_truck/meshes/safeai_Body001.dae"/>
-      </geometry>
-      <material name="black" />
-    </visual>
-    <collision>
-      <!--Wheel/Body001.-->
-      <origin xyz="0.0 0.0 0.0" rpy="0.0 -0.0 0.0"/>
-      <geometry>
-        <mesh filename="package://haul_truck/meshes/safeai_Pad012.dae"/>
-      </geometry>
-      <gazebo>
-        <mu>0.7</mu>
-        <minDepth>0.02</minDepth>
-      </gazebo>
-    </collision>
-    <xacro:sphere_inertial radius="1" mass="2" />
-  </link>
-  <link name="front_left_steering_link">
-    <xacro:box_inertial x="0.1" y="1" z="0.1" mass="1"/>
-  </link>
-  <link name="front_right_steering_link">
-    <xacro:box_inertial x="0.1" y="1" z="0.1" mass="1"/>
-  </link>
-  <joint name="front_left_steering_joint" type="revolute">
-    <parent link="chassis_link" />
-    <child link="front_left_steering_link" />
-    <axis xyz="0 0 1"/>
-    <origin xyz="2.8 3.2 0.6" rpy="0.0 -0.0 0.0"/>
-    <limit lower="-0.4" upper="0.4" effort="10000000" velocity="1000.00"/>
-  </joint>
-  <joint name="front_right_steering_joint" type="revolute">
-    <parent link="chassis_link" />
-    <child link="front_right_steering_link" />
-    <origin xyz="-4.0 3.2 0.6" rpy="0.0 -0.0 0.0"/>
-    <axis xyz="0 0 1"/>
-    <limit lower="-0.4" upper="0.4" effort="10000000" velocity="1000.00"/>
-  </joint>
+  <xacro:wheel name="front_left_wheel_link" />
+  <xacro:wheel name="front_right_wheel_link" />
+  <xacro:wheel name="rear_left_wheel_link" />
+  <xacro:wheel name="rear_right_wheel_link" />
   <joint name="tray_joint" type="fixed">
     <parent link="chassis_link"/>
@@ -180,14 +99,50 @@
     <origin xyz="-3.8 1.0 3.1" rpy="0.0 -0.0 0.0"/>
   </joint>
-  <joint name="front_left_wheel_joint" type="continuous">
-    <parent link="front_left_steering_link"/>
-    <child link="front_left_wheel_link"/>
-    <axis xyz="1 0 0"/>
-  </joint>
-  <joint name="front_right_wheel_joint" type="continuous">
-    <parent link="front_right_steering_link"/>
-    <child link="front_right_wheel_link"/>
-    <axis xyz="1 0 0"/>
-  </joint>
+  <xacro:if value="False">
+    <link name="front_left_steering_link">
+      <xacro:box_inertial x="0.1" y="1" z="0.1" mass="1"/>
+    </link>
+    <link name="front_right_steering_link">
+      <xacro:box_inertial x="0.1" y="1" z="0.1" mass="1"/>
+    </link>
+    <joint name="front_left_steering_joint" type="revolute">
+      <parent link="chassis_link" />
+      <child link="front_left_steering_link" />
+      <axis xyz="0 0 1"/>
+      <origin xyz="2.8 3.2 0.6" rpy="0.0 -0.0 0.0"/>
+      <limit lower="-1.4" upper="1.4" effort="10000000" velocity="1000.00"/>
+    </joint>
+    <joint name="front_right_steering_joint" type="revolute">
+      <parent link="chassis_link" />
+      <child link="front_right_steering_link" />
+      <origin xyz="-4.0 3.2 0.6" rpy="0.0 -0.0 0.0"/>
+      <axis xyz="0 0 1"/>
+      <limit lower="-1.4" upper="1.4" effort="10000000" velocity="1000.00"/>
+    </joint>
+    <joint name="front_left_wheel_joint" type="continuous">
+      <parent link="front_left_steering_link"/>
+      <child link="front_left_wheel_link"/>
+      <axis xyz="1 0 0"/>
+    </joint>
+    <joint name="front_right_wheel_joint" type="continuous">
+      <parent link="front_right_steering_link"/>
+      <child link="front_right_wheel_link"/>
+      <axis xyz="1 0 0"/>
+    </joint>
+  </xacro:if>
+  <xacro:if value="True">
+    <joint name="front_left_wheel_joint" type="continuous">
+      <parent link="chassis_link"/>
+      <child link="front_left_wheel_link"/>
+      <origin xyz="2.8 3.2 0.6" rpy="0.0 -0.0 0.0"/>
+      <axis xyz="1 0 0"/>
+    </joint>
+    <joint name="front_right_wheel_joint" type="continuous">
+      <parent link="chassis_link"/>
+      <child link="front_right_wheel_link"/>
+      <origin xyz="-4.0 3.2 0.6" rpy="0.0 -0.0 0.0"/>
+      <axis xyz="1 0 0"/>
+    </joint>
+  </xacro:if>
   <joint name="rear_left_wheel_joint" type="continuous">
     <parent link="chassis_link"/>
@@ -195,4 +150,5 @@
     <origin xyz="2.8 9.3 0.6" rpy="0.0 -0.0 0.0"/>
     <axis xyz="1 0 0"/>
+    <limit effort="10000000" velocity="1000.00"/>
   </joint>
   <joint name="rear_right_wheel_joint" type="continuous">
@@ -201,4 +157,5 @@
     <origin xyz="-4.0 9.3 0.6" rpy="0.0 -0.0 0.0"/>
     <axis xyz="1 0 0"/>
+    <limit effort="10000000" velocity="1000.00"/>
   </joint>
   <xacro:include filename="$(find haul_truck)/worlds_and_models/haul_truck/lidar_3d_v1.urdf.xacro" />
@@ -212,18 +169,47 @@
       <plugin>ign_ros2_control/IgnitionSystem</plugin>
     </hardware>
-    <joint name="front_left_steering_joint">
-      <command_interface name="position">
-        <param name="min">-0.8727</param>
-        <param name="max">0.8727</param>
-      </command_interface>
-      <state_interface name="position"/>
-    </joint>
-    <joint name="front_right_steering_joint">
-      <command_interface name="position">
-        <param name="min">-0.8727</param>
-        <param name="max">0.8727</param>
-      </command_interface>
-      <state_interface name="position"/>
-    </joint>
+    <xacro:if value="False">
+      <joint name="front_left_steering_joint">
+        <command_interface name="position">
+          <param name="min">-0.8727</param>
+          <param name="max">0.8727</param>
+        </command_interface>
+        <state_interface name="position"/>
+      </joint>
+      <joint name="front_right_steering_joint">
+        <command_interface name="position">
+          <param name="min">-0.8727</param>
+          <param name="max">0.8727</param>
+        </command_interface>
+        <state_interface name="position"/>
+      </joint>
+      <!-- Adding front wheel state interfaces so that their position is given to ros -->
+      <joint name="front_left_wheel_joint">
+        <state_interface name="position"/>
+        <state_interface name="velocity"/>
+      </joint>
+      <joint name="front_right_wheel_joint">
+        <state_interface name="position"/>
+        <state_interface name="velocity"/>
+      </joint>
+    </xacro:if>
+    <xacro:if value="True">
+      <joint name="front_left_wheel_joint">
+        <command_interface name="velocity">
+          <param name="min">-1</param>
+          <param name="max">1</param>
+        </command_interface>
+        <state_interface name="position"/>
+        <state_interface name="velocity"/>
+      </joint>
+      <joint name="front_right_wheel_joint">
+        <command_interface name="velocity">
+          <param name="min">-1</param>
+          <param name="max">1</param>
+        </command_interface>
+        <state_interface name="position"/>
+        <state_interface name="velocity"/>
+      </joint>
+    </xacro:if>
     <joint name="rear_left_wheel_joint">
       <command_interface name="velocity">
@@ -245,5 +231,10 @@
   <gazebo>
     <plugin filename="ign_ros2_control-system" name="ign_ros2_control::IgnitionROS2ControlPlugin">
-      <parameters>$(find haul_truck)/config/ackermann_control.yaml</parameters>
+      <ros>
+        <remapping>/diff_drive_base_controller/odometry:=odom</remapping>
+        <remapping>/diff_drive_base_controller/tf_odometry:=tf</remapping>
+      </ros>
+      <parameters>$(find haul_truck)/config/diffdrive_control.yaml</parameters>
+      <!-- Remapping topics so that mapping system works! -->
     </plugin>
   </gazebo>

File: src/haul_truck/worlds_and_models/haul_truck/lidar_3d_v1.urdf.xacro (robot description, xacro)
@@ -23,26 +23,28 @@
   </joint>
   <gazebo reference="lidar_3d_v1">
-    <sensor name="lidar_2d_v1" type="gpu_ray">
+    <sensor name="lidar_3d_v1" type="gpu_ray">
       <topic>lidar</topic>
-      <ignition_frame_id>lidar_2d_v1</ignition_frame_id>
+      <ignition_frame_id>lidar_3d_v1</ignition_frame_id>
       <pose>0 0 0.0525045525 0 0 0</pose>
       <ray>
         <scan>
           <horizontal>
-            <samples>45</samples>
+            <samples>60</samples>
             <resolution>1</resolution>
-            <min_angle>-0.7</min_angle>
-            <max_angle>0.7</max_angle>
+            <min_angle>-1.41</min_angle>
+            <max_angle>1.14</max_angle>
           </horizontal>
+          <!-- Removing vertical to make slam easier.
           <vertical>
-            <samples>6</samples>
+            <samples>4</samples>
             <resolution>1</resolution>
             <min_angle>-0.52</min_angle>
             <max_angle>0</max_angle>
           </vertical>
+          -->
         </scan>
         <range>
           <min>0.060</min>
-          <max>30</max>
+          <max>100</max>
           <resolution>0.1</resolution>
         </range>

Commit message: Haul truck almost there, but wheels slip too much!

File: src/haul_truck/worlds_and_models/haul_truck/Haul_Truck.urdf.xacro (robot description, xacro)
@@ -42,4 +42,5 @@
     <parent link="base_footprint" />
     <child link="chassis_link" />
+    <origin rpy="0 0 1.5705" />
   </joint>
   <!--Generated by CROSS, a ROS Workbench for FreeCAD (https://github.com/galou/freecad.cross)-->
@@ -56,5 +57,5 @@
       <origin xyz="0.090073 5.25 3.35026" rpy="0.0 -0.0 0.0"/>
       <geometry>
-        <box size="7.6383887394832115 10.500000000000005 4.84423459552541"/>
+        <box size="7.6383887394832115 10.500000000000005 1.84423459552541"/>
       </geometry>
       <gazebo>
@@ -62,5 +63,5 @@
       </gazebo>
     </collision>
-    <xacro:box_inertial_with_origin x="8" y="10" z="3" mass="1">
+    <xacro:box_inertial_with_origin x="8" y="10" z="3" mass="100">
       <origin xyz="0 5 0" rpy="0 0 0" />
     </xacro:box_inertial_with_origin>
@@ -75,4 +76,11 @@
       <material name="red" />
     </visual>
+    <collision>
+      <!--Tray/Body002.-->
+      <origin xyz="0.0 0.0 0.0" rpy="0.0 -0.0 0.0"/>
+      <geometry>
+        <mesh filename="file://$(find haul_truck)/worlds_and_models/haul_truck/meshes/Unnamed_Body002.dae"/>
+      </geometry>
+    </collision>
     <!--
     <collision>
@@ -99,5 +107,5 @@
     <origin xyz="-3.8 1.0 3.1" rpy="0.0 -0.0 0.0"/>
   </joint>
-  <xacro:if value="False">
+  <xacro:if value="True">
     <link name="front_left_steering_link">
       <xacro:box_inertial x="0.1" y="1" z="0.1" mass="1"/>
@@ -111,5 +119,5 @@
       <axis xyz="0 0 1"/>
       <origin xyz="2.8 3.2 0.6" rpy="0.0 -0.0 0.0"/>
-      <limit lower="-1.4" upper="1.4" effort="10000000" velocity="1000.00"/>
+      <limit lower="-0.4" upper="0.4" effort="10000000" velocity="1000.00"/>
     </joint>
     <joint name="front_right_steering_joint" type="revolute">
@@ -118,5 +126,5 @@
       <origin xyz="-4.0 3.2 0.6" rpy="0.0 -0.0 0.0"/>
       <axis xyz="0 0 1"/>
-      <limit lower="-1.4" upper="1.4" effort="10000000" velocity="1000.00"/>
+      <limit lower="-0.4" upper="0.4" effort="10000000" velocity="1000.00"/>
     </joint>
     <joint name="front_left_wheel_joint" type="continuous">
@@ -131,9 +139,10 @@
     </joint>
   </xacro:if>
-  <xacro:if value="True">
+  <xacro:if value="False">
     <joint name="front_left_wheel_joint" type="continuous">
       <parent link="chassis_link"/>
       <child link="front_left_wheel_link"/>
       <origin xyz="2.8 3.2 0.6" rpy="0.0 -0.0 0.0"/>
+      <limit effort="10000000" velocity="1000.00" stiffness="0" dissipation="0"/>
       <axis xyz="1 0 0"/>
     </joint>
@@ -142,4 +151,5 @@
       <child link="front_right_wheel_link"/>
       <origin xyz="-4.0 3.2 0.6" rpy="0.0 -0.0 0.0"/>
+      <limit effort="10000000" velocity="1000.00" stiffness="0" dissipation="0"/>
       <axis xyz="1 0 0"/>
     </joint>
@@ -169,9 +179,9 @@
       <plugin>ign_ros2_control/IgnitionSystem</plugin>
     </hardware>
-    <xacro:if value="False">
+    <xacro:if value="True">
       <joint name="front_left_steering_joint">
         <command_interface name="position">
-          <param name="min">-0.8727</param>
-          <param name="max">0.8727</param>
+          <param name="min">-0.2</param>
+          <param name="max">0.2</param>
         </command_interface>
         <state_interface name="position"/>
@@ -179,6 +189,6 @@
       <joint name="front_right_steering_joint">
         <command_interface name="position">
-          <param name="min">-0.8727</param>
-          <param name="max">0.8727</param>
+          <param name="min">-0.2</param>
+          <param name="max">0.2</param>
         </command_interface>
         <state_interface name="position"/>
@@ -186,13 +196,21 @@
       <!-- Adding front wheel state interfaces so that their position is given to ros -->
       <joint name="front_left_wheel_joint">
+        <command_interface name="velocity">
+          <param name="min">-1</param>
+          <param name="max">1</param>
+        </command_interface>
         <state_interface name="position"/>
         <state_interface name="velocity"/>
       </joint>
       <joint name="front_right_wheel_joint">
+        <command_interface name="velocity">
+          <param name="min">-1</param>
+          <param name="max">1</param>
+        </command_interface>
         <state_interface name="position"/>
         <state_interface name="velocity"/>
       </joint>
     </xacro:if>
-    <xacro:if value="True">
+    <xacro:if value="False">
       <joint name="front_left_wheel_joint">
         <command_interface name="velocity">
@@ -232,8 +250,9 @@
     <plugin filename="ign_ros2_control-system" name="ign_ros2_control::IgnitionROS2ControlPlugin">
       <ros>
-        <remapping>/diff_drive_base_controller/odometry:=odom</remapping>
-        <remapping>/diff_drive_base_controller/tf_odometry:=tf</remapping>
+        <remapping>/ackermann_steering_controller/odometry:=odom</remapping>
+        <remapping>/ackermann_steering_controller/tf_odometry:=tf</remapping>
+        <remapping>/ackermann_steering_controller/reference_unstamped:=cmd_vel</remapping>
       </ros>
-      <parameters>$(find haul_truck)/config/diffdrive_control.yaml</parameters>
+      <parameters>$(find haul_truck)/config/ackermann_control.yaml</parameters>
       <!-- Remapping topics so that mapping system works! -->
     </plugin>
