Commit message: Diff drive working, but still lots of slip

File: src/haul_truck/worlds_and_models/haul_truck/Haul_Truck.urdf.xacro (robot description, xacro)
@@ -1,4 +1,4 @@
 <?xml version="1.0" ?>
-<robot xmlns:xacro="http://www.ros.org/wiki/xacro" name="Haul Truck">
+<robot xmlns:xacro="http://www.ros.org/wiki/xacro" name="haul_truck">
   <material name="red">
     <color rgba="0.816 0.157 0.09 1"/>
@@ -27,14 +27,22 @@
           <mesh filename="file://$(find haul_truck)/worlds_and_models/haul_truck/meshes/safeai_Pad012.dae"/>
         </geometry>
-        <mu>1.0</mu>
-        <mu2>1.0</mu2>
-        <fdir1>0 0 1</fdir1>
-        <slip1>1.0</slip1>
-        <slip2>1.0</slip2>
-        <min_depth>0.5</min_depth>
-        <kp>1e8</kp>
       </collision>
       <xacro:sphere_inertial radius="1" mass="0.2" />
     </link>
+    <gazebo reference="${name}">
+      <surface>
+        <friction>
+          <ode>
+            <mu>1.0</mu>
+            <mu2>1.0</mu2>
+            <fdir1>0 0 1</fdir1>
+            <slip1>0.0</slip1>
+            <slip2>0.0</slip2>
+            <min_depth>0.5</min_depth>
+            <kp>1e8</kp>
+          </ode>
+        </friction>
+      </surface>
+    </gazebo>
   </xacro:macro>
   <link name="base_footprint" />
@@ -107,5 +115,5 @@
     <origin xyz="-3.8 1.0 3.1" rpy="0.0 -0.0 0.0"/>
   </joint>
-  <xacro:if value="True">
+  <xacro:if value="False">
     <link name="front_left_steering_link">
       <xacro:box_inertial x="0.1" y="1" z="0.1" mass="1"/>
@@ -139,5 +147,5 @@
     </joint>
   </xacro:if>
-  <xacro:if value="False">
+  <xacro:if value="True">
     <joint name="front_left_wheel_joint" type="continuous">
       <parent link="chassis_link"/>
@@ -174,4 +182,8 @@
       <render_engine>ogre2</render_engine>
     </plugin>
+    <!-- Publish joints for robot description tf publisher. -->
+    <plugin filename="ignition-gazebo-joint-state-publisher-system" name="ignition::gazebo::systems::JointStatePublisher">
+      <topic>joint_states</topic>
+    </plugin>
   </gazebo>
   <ros2_control name="GazeboSystem" type="system">
@@ -179,5 +191,5 @@
       <plugin>ign_ros2_control/IgnitionSystem</plugin>
     </hardware>
-    <xacro:if value="True">
+    <xacro:if value="False">
       <joint name="front_left_steering_joint">
         <command_interface name="position">
@@ -197,6 +209,6 @@
       <joint name="front_left_wheel_joint">
         <command_interface name="velocity">
-          <param name="min">-1</param>
-          <param name="max">1</param>
+          <param name="min">-0.2</param>
+          <param name="max">0.2</param>
         </command_interface>
         <state_interface name="position"/>
@@ -205,6 +217,6 @@
       <joint name="front_right_wheel_joint">
         <command_interface name="velocity">
-          <param name="min">-1</param>
-          <param name="max">1</param>
+          <param name="min">-0.2</param>
+          <param name="max">0.2</param>
         </command_interface>
         <state_interface name="position"/>
@@ -212,9 +224,9 @@
       </joint>
     </xacro:if>
-    <xacro:if value="False">
+    <xacro:if value="True">
       <joint name="front_left_wheel_joint">
         <command_interface name="velocity">
-          <param name="min">-1</param>
-          <param name="max">1</param>
+          <param name="min">-0.2</param>
+          <param name="max">0.2</param>
         </command_interface>
         <state_interface name="position"/>
@@ -223,6 +235,6 @@
       <joint name="front_right_wheel_joint">
         <command_interface name="velocity">
-          <param name="min">-1</param>
-          <param name="max">1</param>
+          <param name="min">-0.2</param>
+          <param name="max">0.2</param>
         </command_interface>
         <state_interface name="position"/>
@@ -232,6 +244,6 @@
     <joint name="rear_left_wheel_joint">
       <command_interface name="velocity">
-        <param name="min">-1</param>
-        <param name="max">1</param>
+        <param name="min">-0.2</param>
+        <param name="max">0.2</param>
       </command_interface>
       <state_interface name="position"/>
@@ -240,6 +252,6 @@
     <joint name="rear_right_wheel_joint">
       <command_interface name="velocity">
-        <param name="min">-1</param>
-        <param name="max">1</param>
+        <param name="min">-0.2</param>
+        <param name="max">0.2</param>
       </command_interface>
       <state_interface name="position"/>
@@ -250,11 +262,11 @@
     <plugin filename="ign_ros2_control-system" name="ign_ros2_control::IgnitionROS2ControlPlugin">
       <ros>
-        <remapping>/ackermann_steering_controller/odometry:=odom</remapping>
-        <remapping>/ackermann_steering_controller/tf_odometry:=tf</remapping>
-        <remapping>/ackermann_steering_controller/reference_unstamped:=cmd_vel</remapping>
+        <remapping>/diff_drive_base_controller/odometry:=odom</remapping>
+        <remapping>/diff_drive_base_controller/tf_odometry:=tf</remapping>
+        <remapping>/diff_drive_base_controller/cmd_vel_unstamped:=cmd_vel</remapping>
       </ros>
-      <parameters>$(find haul_truck)/config/ackermann_control.yaml</parameters>
-      <!-- Remapping topics so that mapping system works! -->
+      <parameters>$(find haul_truck)/config/diffdrive_control.yaml</parameters>
     </plugin>
+    <!-- Remapping topics so that mapping system works! -->
   </gazebo>
 </robot>

File: src/haul_truck/worlds_and_models/haul_truck/lidar_3d_v1.urdf.xacro (robot description, xacro)
@@ -19,6 +19,6 @@
     <parent link="chassis_link" />
     <child link="lidar_3d_v1" />
-    <!--    <origin rpy="0 0 0" xyz="-1 0 6"/> -->
-    <origin xyz="0.0 0.8 5.7" rpy="0.0 -0.0 -1.57"/>
+    <!--    <origin rpy="0 0 0" xyz="0 0.8 5.6"/> -->
+    <origin xyz="0.0 0.8 8.0" rpy="0.0 -0.0 -1.57"/>
   </joint>
   <gazebo reference="lidar_3d_v1">
@@ -32,6 +32,6 @@
             <samples>60</samples>
             <resolution>1</resolution>
-            <min_angle>-1.41</min_angle>
-            <max_angle>1.14</max_angle>
+            <min_angle>-3.14</min_angle>
+            <max_angle>3.14</max_angle>
           </horizontal>
           <!-- Removing vertical to make slam easier.

Commit message: kr6_working

File: src/haul_truck/worlds_and_models/haul_truck/Haul_Truck.urdf.xacro (robot description, xacro)
@@ -65,5 +65,5 @@
       <origin xyz="0.090073 5.25 3.35026" rpy="0.0 -0.0 0.0"/>
       <geometry>
-        <box size="7.6383887394832115 10.500000000000005 1.84423459552541"/>
+        <box size="7.6383887394832115 10.500000000000005 0.54423459552541"/>
       </geometry>
       <gazebo>
@@ -71,5 +71,5 @@
       </gazebo>
     </collision>
-    <xacro:box_inertial_with_origin x="8" y="10" z="3" mass="100">
+    <xacro:box_inertial_with_origin x="8" y="4" z="3" mass="100">
       <origin xyz="0 5 0" rpy="0 0 0" />
     </xacro:box_inertial_with_origin>
@@ -224,5 +224,5 @@
       </joint>
     </xacro:if>
-    <xacro:if value="True">
+    <xacro:if value="False">
       <joint name="front_left_wheel_joint">
         <command_interface name="velocity">

File: src/veg_bot/worlds_and_models/kuka/kr6r900sixx_macro_simple_geom.xacro (robot description, xacro)
@@ -7,9 +7,4 @@
     <xacro:sphere_inertial radius="1" mass="2" />
   </xacro:macro>
-  <link name="world" />
-  <joint name="world_link" type="fixed">
-    <parent link="world" />
-    <child link="base_link" />
-  </joint>
   <xacro:macro name="kuka_kr6r900sixx" params="prefix">
     <link name="${prefix}base_link">
@@ -22,7 +17,7 @@
       </visual>
       <collision>
-        <origin xyz="0 0 0" rpy="0 0 0"/>
-        <geometry>
-          <mesh filename="file://$(find veg_bot)/worlds_and_models/kuka/meshes/kr6_agilus/collision/base_link.stl" />
+        <origin xyz="-0.01 0 0" rpy="0 0 0"/>
+        <geometry>
+          <box size="0.33 0.21 0.4"/>
         </geometry>
       </collision>
@@ -40,5 +35,5 @@
         <origin xyz="0 0 0" rpy="0 0 0"/>
         <geometry>
-          <mesh filename="file://$(find veg_bot)/worlds_and_models/kuka/meshes/kr6_agilus/collision/link_1.stl" />
+          <box size="0.24 0.28 0.27" />
         </geometry>
       </collision>
@@ -54,7 +49,7 @@
       </visual>
       <collision>
-        <origin xyz="0 0 0" rpy="0 0 0"/>
-        <geometry>
-          <mesh filename="file://$(find veg_bot)/worlds_and_models/kuka/meshes/kr6r900sixx/collision/link_2.stl" />
+        <origin xyz="0.1 0 0" rpy="0 0 0"/>
+        <geometry>
+          <box size="0.63 0.25 0.18" />
         </geometry>
       </collision>
@@ -70,7 +65,7 @@
       </visual>
       <collision>
-        <origin xyz="0 0 0" rpy="0 0 0"/>
-        <geometry>
-          <mesh filename="file://$(find veg_bot)/worlds_and_models/kuka/meshes/kr6_agilus/collision/link_3.stl" />
+        <origin xyz="0.0 0 0" rpy="0 0 0"/>
+        <geometry>
+          <box size="0.19 0.13 0.17" />
         </geometry>
       </collision>
@@ -86,7 +81,7 @@
       </visual>
       <collision>
-        <origin xyz="0 0 0" rpy="0 0 0"/>
-        <geometry>
-          <mesh filename="file://$(find veg_bot)/worlds_and_models/kuka/meshes/kr6r900sixx/collision/link_4.stl" />
+        <origin xyz="0.2 0 0" rpy="0 0 0"/>
+        <geometry>
+          <box size="0.45 0.12 0.13" />
         </geometry>
       </collision>
@@ -102,7 +97,7 @@
       </visual>
       <collision>
-        <origin xyz="0 0 0" rpy="0 0 0"/>
-        <geometry>
-          <mesh filename="file://$(find veg_bot)/worlds_and_models/kuka/meshes/kr6_agilus/collision/link_5.stl" />
+        <origin xyz="0.01 0 0" rpy="0 0 0"/>
+        <geometry>
+          <box size="0.10 0.1 0.1" />
         </geometry>
       </collision>
@@ -120,5 +115,5 @@
         <origin xyz="0 0 0" rpy="0 0 0"/>
         <geometry>
-          <mesh filename="file://$(find veg_bot)/worlds_and_models/kuka/meshes/kr6_agilus/collision/link_6.stl" />
+          <box size="0.013 0.040 0.04" />
         </geometry>
       </collision>
@@ -132,5 +127,5 @@
       <child link="${prefix}link_1"/>
       <axis xyz="0 0 -1"/>
-      <limit effort="1000" lower="${-radians(170)}" upper="${radians(170)}" velocity="${radians(360)}"/>
+      <limit effort="0" lower="${-radians(170)}" upper="${radians(170)}" velocity="${radians(360)}"/>
     </joint>
     <joint name="${prefix}joint_a2" type="revolute">
@@ -139,5 +134,5 @@
       <child link="${prefix}link_2"/>
       <axis xyz="0 1 0"/>
-      <limit effort="1000" lower="${-radians(190)}" upper="${radians(45)}" velocity="${radians(300)}"/>
+      <limit effort="0" lower="${-radians(190)}" upper="${radians(45)}" velocity="${radians(300)}"/>
     </joint>
     <joint name="${prefix}joint_a3" type="revolute">
@@ -146,5 +141,5 @@
       <child link="${prefix}link_3"/>
       <axis xyz="0 1 0"/>
-      <limit effort="1000" lower="${-radians(120)}" upper="${radians(156)}" velocity="${radians(360)}"/>
+      <limit effort="0" lower="${-radians(120)}" upper="${radians(156)}" velocity="${radians(360)}"/>
     </joint>
     <joint name="${prefix}joint_a4" type="revolute">
@@ -153,5 +148,5 @@
       <child link="${prefix}link_4"/>
       <axis xyz="-1 0 0"/>
-      <limit effort="1000" lower="${-radians(185)}" upper="${radians(185)}" velocity="${radians(381)}"/>
+      <limit effort="0" lower="${-radians(185)}" upper="${radians(185)}" velocity="${radians(381)}"/>
     </joint>
     <joint name="${prefix}joint_a5" type="revolute">
@@ -160,5 +155,5 @@
       <child link="${prefix}link_5"/>
       <axis xyz="0 1 0"/>
-      <limit effort="1000" lower="${-radians(120)}" upper="${radians(120)}" velocity="${radians(388)}"/>
+      <limit effort="0" lower="${-radians(120)}" upper="${radians(120)}" velocity="${radians(388)}"/>
     </joint>
     <joint name="${prefix}joint_a6" type="revolute">
@@ -167,5 +162,5 @@
       <child link="${prefix}link_6"/>
       <axis xyz="-1 0 0"/>
-      <limit effort="1000" lower="${-radians(350)}" upper="${radians(350)}" velocity="${radians(615)}"/>
+      <limit effort="0" lower="${-radians(350)}" upper="${radians(350)}" velocity="${radians(615)}"/>
     </joint>
     <joint name="${prefix}joint_a6-flange" type="fixed">
@@ -202,10 +197,4 @@
       <origin xyz="0 0 0" rpy="0 0 0"/>
     </joint>
-    <link name="tool_tip" />
-    <joint name="suction_tool_tip" type="fixed">
-      <parent link="tool0"/>
-      <child link="tool_tip"/>
-      <origin xyz="0.32 0 0" />
-    </joint>
   </xacro:macro>
 </robot>

Commit message: Adding collision property to wheels

File: src/haul_truck/worlds_and_models/haul_truck/Haul_Truck.urdf.xacro (robot description, xacro)
@@ -31,17 +31,19 @@
     </link>
     <gazebo reference="${name}">
-      <surface>
-        <friction>
-          <ode>
-            <mu>1.0</mu>
-            <mu2>1.0</mu2>
-            <fdir1>0 0 1</fdir1>
-            <slip1>0.0</slip1>
-            <slip2>0.0</slip2>
-            <min_depth>0.5</min_depth>
-            <kp>1e8</kp>
-          </ode>
-        </friction>
-      </surface>
+      <collision>
+        <surface>
+          <friction>
+            <ode>
+              <mu>1.0</mu>
+              <mu2>1.0</mu2>
+              <fdir1>0 0 1</fdir1>
+              <slip1>0.0</slip1>
+              <slip2>0.0</slip2>
+              <min_depth>0.5</min_depth>
+              <kp>1e8</kp>
+            </ode>
+          </friction>
+        </surface>
+      </collision>
     </gazebo>
   </xacro:macro>
