Commit message: Tuned Gazebo sim of Scorpion

File: src/freecad_scorpion/urdf/Robot.urdf (robot description, URDF)
Before this commit: robot Robot, 12 links, 11 joints
Links:
- removed link chasis_link
- removed link left_wheel_1_link
- removed link left_wheel_2_link
- removed link left_wheel_3_link
- removed link left_wheel_4_link
- removed link right_wheel_1_link
- removed link right_wheel_2_link
- removed link right_wheel_3_link
- removed link right_wheel_4_link
- removed link tail1_link
- removed link tail2_link
- removed link tail3_link
- added link chassis_link, mass 0.0; visual mesh filename=package://freecad_scorpion/meshes/Unnamed_chassis_body.dae
- added link left_wheel_1, mass 0.0; visual mesh filename=package://freecad_scorpion/meshes/Unnamed_wheel_body.dae
- added link left_wheel_2, mass 0.0; visual mesh filename=package://freecad_scorpion/meshes/Unnamed_wheel_body.dae
- added link left_wheel_3, mass 0.0; visual mesh filename=package://freecad_scorpion/meshes/Unnamed_wheel_body.dae
- added link right_wheel_1, mass 0.0; visual mesh filename=package://freecad_scorpion/meshes/Unnamed_wheel_body.dae
- added link right_wheel_2, mass 0.0; visual mesh filename=package://freecad_scorpion/meshes/Unnamed_wheel_body.dae
- added link right_wheel_3, mass 0.0; visual mesh filename=package://freecad_scorpion/meshes/Unnamed_wheel_body.dae
- added link tail_link1, mass 0.0; visual mesh filename=package://freecad_scorpion/meshes/Unnamed_tail1_body.dae
- added link tail_link2, mass 0.0; visual mesh filename=package://freecad_scorpion/meshes/Unnamed_tail2_body.dae
- added link tail_link3, mass 0.0; visual mesh filename=package://freecad_scorpion/meshes/Unnamed_tail3_body.dae
Joints:
- removed joint joint1
- removed joint joint2
- removed joint joint3
- removed joint left_wheel_j1
- removed joint left_wheel_j2
- removed joint left_wheel_j3
- removed joint left_wheel_j4
- removed joint right_wheel_j1
- removed joint right_wheel_j2
- removed joint right_wheel_j3
- removed joint right_wheel_j4
- added joint joint_1: type revolute, parent chassis_link, child tail_link1, origin xyz=0.19 0.0 0.05 rpy=0.0 0.7853981633974484 0.0, axis 0 1 0, limit lower=0.0 upper=3.141592653589793 effort=10.0 velocity=0.0
- added joint joint_2: type revolute, parent tail_link1, child tail_link2, origin xyz=-0.065 0.0 -0.008 rpy=0.0 -0.0 0.0, axis 0 0 1, limit lower=-1.5707963267948966 upper=1.5707963267948966 effort=10.0 velocity=0.17453292519943295
- added joint joint_3: type revolute, parent tail_link2, child tail_link3, origin xyz=-0.046 0.0 0.0 rpy=0.0 -0.0 0.0, axis 0 1 0, limit lower=-1.5707963267948966 upper=1.5707963267948966 effort=10.0 velocity=0.017453292519943295
- added joint left_wheel_3_joint: type continuous, parent chassis_link, child left_wheel_3, origin xyz=0.16 -0.033 0.015 rpy=0.0 -0.0 0.0, axis 0 1 0, limit lower=0.0 upper=0.0 effort=10.0 velocity=0.001
- added joint left_wheel_joint1: type continuous, parent chassis_link, child left_wheel_1, origin xyz=0.02 -0.033 0.015 rpy=0.0 -0.0 0.0, axis 0 1 0, limit lower=0.0 upper=0.0 effort=10.0 velocity=0.001
- added joint left_wheel_joint2: type continuous, parent chassis_link, child left_wheel_2, origin xyz=0.09 -0.033 0.015 rpy=0.0 -0.0 0.0, axis 0 1 0, limit lower=0.0 upper=0.0 effort=10.0 velocity=0.001
- added joint right_wheel_3_joint: type continuous, parent chassis_link, child right_wheel_3, origin xyz=0.16 0.033 0.015 rpy=0.0 -0.0 0.0, axis 0 1 0, limit lower=0.0 upper=0.0 effort=10.0 velocity=0.001
- added joint right_wheel_joint1: type continuous, parent chassis_link, child right_wheel_1, origin xyz=0.02 0.033 0.015 rpy=0.0 -0.0 0.0, axis 0 1 0, limit lower=0.0 upper=0.0 effort=10.0 velocity=0.001
- added joint right_wheel_joint2: type continuous, parent chassis_link, child right_wheel_2, origin xyz=0.09 0.033 0.015 rpy=0.0 -0.0 0.0, axis 0 1 0, limit lower=0.0 upper=0.0 effort=10.0 velocity=0.001

Commit message: Adding freecad design files

File: src/freecad_scorpion/urdf/Robot.urdf (robot description, URDF)
Before this commit: robot Robot, 10 links, 9 joints
Joints:
- joint right_wheel_3_joint: axis 0 1 0 -> 0 0 1
